File: power-and-uart.sch (KiCad schematic (older format))
At the start: 41 parts, among them J1002 USB_miniB, J1003 USB_C_Receptacle_USB2.0, U1001 USB3740B-AI9, U1002 UTC2000, U1003 FT232RL, U1004 74LVC1G00, U1005 SC185

Commit message: use special +5/+3V3 labels with more specific net names
This allows easier integration since these are global labels
and using more specific names helps avoiding clashes.

The labels are stored in the 'rescue' library.

Strangely: the same trick did not work for GND. Kicad always
insists the net name remains 'GND' (it does work, however if
a new schematic is created - then the different net name for
GND 'sticks').
Connections:
- net VIN_3V3 is gone; now on net +3V3_PWR_OUT: C1006.1, C1008.1, L1001.1, U1005.10 (VOUT)
- net +3V3 renamed +3V3_PWR_OUT
- net +5V renamed +5V_PWR_OUT
Changed lines of the file:
@@
 	4300 6800 4300 7300
 $Comp
-L power:+3V3 #PWR?
+L power-test-module-rescue:+3V3 #PWR?
 U 1 1 5C383ABB
 P 5300 5800
@@
 $EndComp
 $Comp
-L power:+5V #PWR?
+L power-test-module-rescue:+5V #PWR?
 U 1 1 5C383AC1
 P 5500 5800
@@
 	4600 6500 3150 6500
 $Comp
-L power:+5V #PWR?
+L power-test-module-rescue:+5V #PWR?
 U 1 1 5C383B30
 P 2750 6200
@@
 	3300 6200 4300 6200
 $Comp
-L power:+5V #PWR?
+L power-test-module-rescue:+5V #PWR?
 U 1 1 5C383B43
 P 3900 5950
@@
 Wire Wire Line
 	3000 5950 3050 5950
-$Comp
-L power:PWR_FLAG #FLG?
-U 1 1 5C3CF027
-P 8100 1000
-AR Path="/5C3C60AE/5C3CF027" Ref="#FLG?"  Part="1"
-AR Path="/5C3CF027" Ref="#FLG?"  Part="1"
-AR Path="/5C4CE703/5C3CF027" Ref="#FLG?"  Part="1"
-F 0 "#FLG?" H 8100 1075 50  0001 C CNN
-F 1 "PWR_FLAG" H 8100 1174 50  0000 C CNN
-F 2 "" H 8100 1000 50  0001 C CNN
-F 3 "~" H 8100 1000 50  0001 C CNN
-	1    8100 1000
-	1    0    0    1
-$EndComp
-Connection ~ 8100 1000
-Wire Wire Line
-	8100 1000 8300 1000
 $Comp
 L Device:L_Core_Ferrite L?
@@
 Connection ~ 7200 1000
 $Comp
-L power:+5V #PWR?
+L power-test-module-rescue:+5V #PWR?
 U 1 1 5C3CF0BE
 P 5050 1950
@@
 $EndComp
 $Comp
-L power:+5V #PWR?
+L power-test-module-rescue:+5V #PWR?
 U 1 1 5C3CF10A
 P 4700 3750
@@
 	4100 3200 4150 3200
 $Comp
-L power:+5V #PWR?
+L power-test-module-rescue:+5V #PWR?
 U 1 1 5C3CF114
 P 4150 3200
@@
 $EndComp
 $Comp
-L power:+5V #PWR?
+L power-test-module-rescue:+5V #PWR?
 U 1 1 5C3CF17B
 P 6850 3200
@@
 Connection ~ 5550 3650
 $Comp
-L power:+5V #PWR?
+L power-test-module-rescue:+5V #PWR?
 U 1 1 5C42AC0F
 P 5350 3600
@@
 	5800 4200 5800 4600
 $Comp
-L power:+5V #PWR?
+L power-test-module-rescue:+5V #PWR?
 U 1 1 5C4ED32E
 P 4650 5100
@@
 Text Notes 6400 5200 0    50   ~ 0
 Upgrades:\n- use LVC1G10 (3 input nand) and evaluate\n  LEG# with additional input/jumper\n- add USB mux option (e.g. TS3USB221)
-$Comp
-L trigbox:VIN_3V3 #PWR?
-U 1 1 60D3740A
-P 8300 1000
-F 0 "#PWR?" H 8300 850 50  0001 C CNN
-F 1 "VIN_3V3" H 8315 1173 50  0000 C CNN
-F 2 "" H 8300 1000 50  0001 C CNN
-F 3 "" H 8300 1000 50  0001 C CNN
-	1    8300 1000
-	1    0    0    -1
-$EndComp
-Wire Wire Line
-	7200 1000 8100 1000
 Wire Wire Line
 	5700 2150 5700 2700
@@
 $EndComp
 NoConn ~ 2700 2700
+$Comp
+L power-test-module-rescue:+3V3 #PWR?
+U 1 1 60DA0D30
+P 8300 1000
+AR Path="/5BE73D36/60DA0D30" Ref="#PWR?"  Part="1"
+AR Path="/5C1147CA/60DA0D30" Ref="#PWR?"  Part="1"
+AR Path="/60DA0D30" Ref="#PWR?"  Part="1"
+AR Path="/5C4CE703/60DA0D30" Ref="#PWR?"  Part="1"
+F 0 "#PWR?" H 8300 850 50  0001 C CNN
+F 1 "+3V3" H 8315 1173 50  0000 C CNN
+F 2 "" H 8300 1000 50  0001 C CNN
+F 3 "" H 8300 1000 50  0001 C CNN
+	1    8300 1000
+	1    0    0    -1
+$EndComp
+Wire Wire Line
+	7200 1000 8300 1000
 $EndSCHEMATC

Commit message: re-annotated for merging; updated PCB
Parts:
- renumbered C1001 to C1101, C1002 to C1102, C1003 to C1103, C1004 to C1104, C1005 to C1105, C1006 to C1106, C1007 to C1107, C1008 to C1108, D1001 to D1101, D1002 to D1102, D1003 to D1103, FL1001 to FL1101, FL1002 to FL1102, J1002 to J1101, J1003 to J1102, JP1001 to JP1101, JP1002 to JP1102, L1001 to L1101, R1001 to R1101, R1002 to R1102, R1003 to R1103, R1004 to R1104, R1005 to R1105, R1006 to R1106, R1007 to R1107, R1008 to R1108, R1009 to R1109, R1010 to R1110, R1011 to R1111, R1012 to R1112, R1013 to R1113, R1014 to R1114, R1015 to R1115, R1016 to R1116, R1017 to R1117, R1018 to R1118, U1001 to U1101, U1002 to U1102, U1003 to U1103, U1004 to U1104, U1005 to U1105
