File: power-and-uart.sch (KiCad schematic (older format))
At the start: 41 parts, among them J1002 USB_miniB, J1003 USB_C_Receptacle_USB2.0, U1001 USB3740B-AI9, U1002 UTC2000, U1003 FT232RL, U1004 74LVC1G00, U1005 SC185

Commit message: added part numbers for EMI filter + LEDs;
Also changed reset pullup from 4k7 to 5k1 (for sake of fewer different values)
Parts:
- D1001, D1002: Manufacturer (none) -> Wurth; Part (none) -> 150060GS75000
- D1003: Manufacturer (none) -> Wurth; Part (none) -> 150060RS75000
- FL1001, FL1002: Manufacturer (none) -> Wurth; Part (none) -> 744231371
- R1010: value R4k7 -> 5k1; symbol trigbox:R4k7 -> Device:R_Small
Changed lines of the file:
@@
 F 2 "proj_footprints:WE_CNSW" V 1600 7540 50  0001 C CNN
 F 3 "https://www.digikey.com/catalog/en/partgroup/we-cnsw-we-cnsw-hf/22783?mpart=744231371&vendor=732" H 1600 7687 50  0001 C CNN
+F 4 "744231371" H 1600 7500 50  0001 C CNN "Part"
+F 5 "Wurth" H 1600 7500 50  0001 C CNN "Manufacturer"
 	1    1600 7500
 	1    0    0    1
@@
 	4300 7500 4600 7500
 $Comp
-L trigbox:R4k7 R1010
+L Device:R_Small R1010
 U 1 1 5C383AEE
 P 4300 6700
 F 0 "R1010" H 4359 6730 50  0000 L CNN
-F 1 "R4k7" H 4359 6654 30  0000 L CNN
+F 1 "5k1" H 4359 6654 50  0000 L CNN
 F 2 "Resistor_SMD:R_0603_1608Metric" H 4300 6700 50  0001 C CNN
 F 3 "~" H 4300 6700 50  0001 C CNN
@@
 F 2 "proj_footprints:WE_CNSW" V 1850 6490 50  0001 C CNN
 F 3 "https://www.digikey.com/catalog/en/partgroup/we-cnsw-we-cnsw-hf/22783?mpart=744231371&vendor=732" H 1850 6637 50  0001 C CNN
+F 4 "744231371" H 1850 6450 50  0001 C CNN "Part"
+F 5 "Wurth" H 1850 6450 50  0001 C CNN "Manufacturer"
 	1    1850 6450
 	1    0    0    -1
@@
 F 2 "LED_SMD:LED_0603_1608Metric" H 6500 3500 50  0001 C CNN
 F 3 "~" H 6500 3500 50  0001 C CNN
+F 4 "150060RS75000" H 6500 3500 50  0001 C CNN "Part"
+F 5 "Wurth" H 6500 3500 50  0001 C CNN "Manufacturer"
 	1    6500 3500
 	1    0    0    -1
@@
 F 2 "LED_SMD:LED_0603_1608Metric" H 5000 4550 50  0001 C CNN
 F 3 "~" H 5000 4550 50  0001 C CNN
+F 4 "150060GS75000" H 5000 4550 50  0001 C CNN "Part"
+F 5 "Wurth" H 5000 4550 50  0001 C CNN "Manufacturer"
 	1    5000 4550
 	0    -1   -1   0
@@
 F 2 "LED_SMD:LED_0603_1608Metric" H 5350 4550 50  0001 C CNN
 F 3 "~" H 5350 4550 50  0001 C CNN
+F 4 "150060GS75000" H 5350 4550 50  0001 C CNN "Part"
+F 5 "Wurth" H 5350 4550 50  0001 C CNN "Manufacturer"
 	1    5350 4550
 	0    -1   -1   0

Commit message: added/updated part number of inductor
Parts:
- L1001: Manufacturer TOKO -> Sumida; Model FDV0530S-1R0 -> (none); Part (none) -> CDMC6D28NP-1R0MC
Changed lines of the file:
@@
 F 2 "proj_footprints:L_CDMC6D28" H 6800 1000 50  0001 C CNN
 F 3 "~" H 6800 1000 50  0001 C CNN
-F 4 "TOKO" V 6800 1000 50  0001 C CNN "Manufacturer"
-F 5 "FDV0530S-1R0" V 6800 1000 50  0001 C CNN "Model"
+F 4 "Sumida" V 6800 1000 50  0001 C CNN "Manufacturer"
+F 5 "CDMC6D28NP-1R0MC " V 6800 1000 50  0001 C CNN "Part"
 	1    6800 1000
 	0    1    1    0
