File: power-and-uart.sch (KiCad schematic (older format))
At the start: 41 parts, among them J1101 USB_miniB, J1102 USB_C_Receptacle_USB2.0, U1101 USB3740B-AI9, U1102 UTC2000, U1103 FT232RL, U1104 74LVC1G00, U1105 SC185

Commit message: various mods to adapt to dev-board
Parts:
- D1101, D1102: Manufacturer (none) -> Wurth; Part (none) -> 150060GS75000
- D1103: Manufacturer (none) -> Wurth; Part (none) -> 150060RS75000
- R1102, R1103, R1116, R1117: value R100k -> 100k; symbol trigbox:R100k -> Device:R_Small
- R1105, R1106, R1107, R1108, R1111: value R10k -> 10k
- R1110: value R4k7 -> 5k1; symbol trigbox:R4k7 -> Device:R_Small
Changed lines of the file:
@@
 $Descr USLetter 11000 8500
 encoding utf-8
-Sheet 6 11
+Sheet 6 12
 Title ""
 Date ""
@@
 P 4300 7400
 F 0 "R1111" H 4359 7430 50  0000 L CNN
-F 1 "R10k" H 4359 7354 30  0000 L CNN
+F 1 "10k" H 4359 7354 30  0000 L CNN
 F 2 "Resistor_SMD:R_0603_1608Metric" H 4300 7400 50  0001 C CNN
 F 3 "~" H 4300 7400 50  0001 C CNN
@@
 	4300 7500 4600 7500
 $Comp
-L trigbox:R4k7 R1110
+L Device:R_Small R1110
 U 1 1 5C383AEE
 P 4300 6700
 F 0 "R1110" H 4359 6730 50  0000 L CNN
-F 1 "R4k7" H 4359 6654 30  0000 L CNN
+F 1 "5k1" H 4359 6654 30  0000 L CNN
 F 2 "Resistor_SMD:R_0603_1608Metric" H 4300 6700 50  0001 C CNN
 F 3 "~" H 4300 6700 50  0001 C CNN
@@
 	3900 5950 3550 5950
 $Comp
-L trigbox:R100k R1102
+L Device:R_Small R1102
 U 1 1 5C383B4A
 P 3300 6700
 F 0 "R1102" H 3241 6670 50  0000 R CNN
-F 1 "R100k" H 3241 6746 30  0000 R CNN
+F 1 "100k" H 3241 6746 30  0000 R CNN
 F 2 "Resistor_SMD:R_0603_1608Metric" H 3300 6700 50  0001 C CNN
 F 3 "~" H 3300 6700 50  0001 C CNN
@@
 $EndComp
 $Comp
-L trigbox:R100k R1103
+L Device:R_Small R1103
 U 1 1 5C383B51
 P 3300 6900
 F 0 "R1103" H 3241 6870 50  0000 R CNN
-F 1 "R100k" H 3241 6946 30  0000 R CNN
+F 1 "100k" H 3241 6946 30  0000 R CNN
 F 2 "Resistor_SMD:R_0603_1608Metric" H 3300 6900 50  0001 C CNN
 F 3 "~" H 3300 6900 50  0001 C CNN
@@
 AR Path="/5C4CE703/5C3CF043" Ref="C1104"  Part="1"
 AR Path="/60DAA393/5C4CE703/5C3CF043" Ref="C1104"  Part="1"
-F 0 "C1104" H 4800 2100 50  0000 L CNN
-F 1 "22uF_lo_ESR" H 4500 2000 50  0000 L CNN
+F 0 "C1104" H 4750 2200 50  0000 L CNN
+F 1 "22uF_lo_ESR" H 4600 2000 50  0000 L CNN
 F 2 "Capacitor_SMD:C_1812_4532Metric" H 5088 1950 50  0001 C CNN
 F 3 "https://product.tdk.com/info/en/documents/chara_sheet/C4532X7R1E226M250KC.pdf" H 5050 2100 50  0001 C CNN
@@
 AR Path="/5C4CE703/5C3CF04C" Ref="C1105"  Part="1"
 AR Path="/60DAA393/5C4CE703/5C3CF04C" Ref="C1105"  Part="1"
-F 0 "C1105" H 5850 2600 50  0000 R CNN
+F 0 "C1105" H 6000 2600 50  0000 R CNN
 F 1 "100nF_603" H 6150 2500 50  0000 R CNN
 F 2 "Capacitor_SMD:C_0603_1608Metric" H 5638 2400 50  0001 C CNN
@@
 AR Path="/5C4CE703/5C3CF0FC" Ref="R1108"  Part="1"
 AR Path="/60DAA393/5C4CE703/5C3CF0FC" Ref="R1108"  Part="1"
-F 0 "R1108" H 4250 3350 50  0000 L CNN
-F 1 "R10k" H 4259 3254 30  0000 L CNN
+F 0 "R1108" H 4300 3400 50  0000 L CNN
+F 1 "10k" H 4259 3254 30  0000 L CNN
 F 2 "Resistor_SMD:R_0603_1608Metric" H 4200 3300 50  0001 C CNN
 F 3 "~" H 4200 3300 50  0001 C CNN
@@
 AR Path="/5C4CE703/5C3CF103" Ref="R1107"  Part="1"
 AR Path="/60DAA393/5C4CE703/5C3CF103" Ref="R1107"  Part="1"
-F 0 "R1107" H 3900 3350 50  0000 L CNN
-F 1 "R10k" H 3900 3250 30  0000 L CNN
+F 0 "R1107" H 3800 3400 50  0000 L CNN
+F 1 "10k" H 3900 3250 30  0000 L CNN
 F 2 "Resistor_SMD:R_0603_1608Metric" H 4100 3300 50  0001 C CNN
 F 3 "~" H 4100 3300 50  0001 C CNN
@@
 AR Path="/60DAA393/5C4CE703/5C3CF124" Ref="R1105"  Part="1"
 F 0 "R1105" H 3250 3550 50  0000 L CNN
-F 1 "R10k" H 3300 3450 30  0000 L CNN
+F 1 "10k" H 3300 3450 30  0000 L CNN
 F 2 "Resistor_SMD:R_0603_1608Metric" H 3450 3500 50  0001 C CNN
 F 3 "~" H 3450 3500 50  0001 C CNN
@@
 AR Path="/60DAA393/5C4CE703/5C3CF12B" Ref="R1106"  Part="1"
 F 0 "R1106" H 3600 3550 50  0000 L CNN
-F 1 "R10k" H 3609 3454 30  0000 L CNN
+F 1 "10k" H 3609 3454 30  0000 L CNN
 F 2 "Resistor_SMD:R_0603_1608Metric" H 3550 3500 50  0001 C CNN
 F 3 "~" H 3550 3500 50  0001 C CNN
@@
 AR Path="/5C4CE703/5C3CF15A" Ref="C1103"  Part="1"
 AR Path="/60DAA393/5C4CE703/5C3CF15A" Ref="C1103"  Part="1"
-F 0 "C1103" V 4600 3850 50  0000 C CNN
+F 0 "C1103" V 4600 3900 50  0000 C CNN
 F 1 "100nF_603" V 4700 3950 50  0000 C CNN
 F 2 "Capacitor_SMD:C_0603_1608Metric" H 4888 3650 50  0001 C CNN
@@
 	4100 4600 4100 4750
 $Comp
-L trigbox:R100k R?
+L Device:R_Small R?
 U 1 1 5C3CF184
 P 5550 3750
@@
 AR Path="/5C4CE703/5C3CF184" Ref="R1116"  Part="1"
 AR Path="/60DAA393/5C4CE703/5C3CF184" Ref="R1116"  Part="1"
-F 0 "R1116" H 5350 3800 50  0000 L CNN
-F 1 "R100k" H 5350 3700 30  0000 L CNN
+F 0 "R1116" H 5400 3950 50  0000 L CNN
+F 1 "100k" H 5350 3700 30  0000 L CNN
 F 2 "Resistor_SMD:R_0603_1608Metric" H 5550 3750 50  0001 C CNN
 F 3 "~" H 5550 3750 50  0001 C CNN
@@
 Wire Wire Line
 	6350 3500 6350 4150
-$Comp
-L Device:LED D?
-U 1 1 5C3CF191
-P 6500 3500
-AR Path="/5C3C60AE/5C3CF191" Ref="D?"  Part="1"
-AR Path="/5C3CF191" Ref="D?"  Part="1"
-AR Path="/5C4CE703/5C3CF191" Ref="D1103"  Part="1"
-AR Path="/60DAA393/5C4CE703/5C3CF191" Ref="D1103"  Part="1"
-F 0 "D1103" H 6491 3716 50  0000 C CNN
-F 1 "LED" H 6491 3625 50  0000 C CNN
-F 2 "LED_SMD:LED_0603_1608Metric" H 6500 3500 50  0001 C CNN
-F 3 "~" H 6500 3500 50  0001 C CNN
-	1    6500 3500
-	1    0    0    -1
-$EndComp
-Connection ~ 6350 3500
 Wire Wire Line
 	2700 2200 2700 2250
@@
 Alt: CDMC6D28NP-1RØMC
 $Comp
-L trigbox:R100k R?
+L Device:R_Small R?
 U 1 1 5C3EC942
 P 5800 3750
@@
 AR Path="/5C4CE703/5C3EC942" Ref="R1117"  Part="1"
 AR Path="/60DAA393/5C4CE703/5C3EC942" Ref="R1117"  Part="1"
-F 0 "R1117" H 5600 3800 50  0000 L CNN
-F 1 "R100k" H 5600 3700 30  0000 L CNN
+F 0 "R1117" H 5750 3950 50  0000 L CNN
+F 1 "100k" H 5600 3700 30  0000 L CNN
 F 2 "Resistor_SMD:R_0603_1608Metric" H 5800 3750 50  0001 C CNN
 F 3 "~" H 5800 3750 50  0001 C CNN
@@
 F 2 "LED_SMD:LED_0603_1608Metric" H 5000 4550 50  0001 C CNN
 F 3 "~" H 5000 4550 50  0001 C CNN
+F 4 "Wurth" H 5000 4550 50  0001 C CNN "Manufacturer"
+F 5 " 150060GS75000 " H 5000 4550 50  0001 C CNN "Part"
 	1    5000 4550
 	0    -1   -1   0
@@
 F 2 "LED_SMD:LED_0603_1608Metric" H 5350 4550 50  0001 C CNN
 F 3 "~" H 5350 4550 50  0001 C CNN
+F 4 "Wurth" H 5350 4550 50  0001 C CNN "Manufacturer"
+F 5 " 150060GS75000 " H 5350 4550 50  0001 C CNN "Part"
 	1    5350 4550
 	0    -1   -1   0
@@
 AR Path="/5C4CE703/5C393D05" Ref="C1102"  Part="1"
 AR Path="/60DAA393/5C4CE703/5C393D05" Ref="C1102"  Part="1"
-F 0 "C1102" H 4615 2146 50  0000 L CNN
-F 1 "100nF_603" H 4615 2055 50  0000 L CNN
+F 0 "C1102" H 4150 2200 50  0000 L CNN
+F 1 "100nF_603" H 4050 2000 50  0000 L CNN
 F 2 "Capacitor_SMD:C_0603_1608Metric" H 4538 1950 50  0001 C CNN
 F 3 "~" H 4500 2100 50  0001 C CNN
@@
 Wire Wire Line
 	6200 6200 6550 6200
-Text Notes 6400 5200 0    50   ~ 0
-Upgrades:\n- use LVC1G10 (3 input nand) and evaluate\n  LEG# with additional input/jumper\n- add USB mux option (e.g. TS3USB221)
 Wire Wire Line
 	5700 2150 5700 2700
@@
 Wire Wire Line
 	7200 1000 8300 1000
+Connection ~ 6350 3500
+$Comp
+L Device:LED D?
+U 1 1 5C3CF191
+P 6500 3500
+AR Path="/5C3C60AE/5C3CF191" Ref="D?"  Part="1"
+AR Path="/5C3CF191" Ref="D?"  Part="1"
+AR Path="/5C4CE703/5C3CF191" Ref="D1103"  Part="1"
+AR Path="/60DAA393/5C4CE703/5C3CF191" Ref="D1103"  Part="1"
+F 0 "D1103" H 6491 3716 50  0000 C CNN
+F 1 "LED" H 6491 3625 50  0000 C CNN
+F 2 "LED_SMD:LED_0603_1608Metric" H 6500 3500 50  0001 C CNN
+F 3 "~" H 6500 3500 50  0001 C CNN
+F 4 "Wurth" H 6500 3500 50  0001 C CNN "Manufacturer"
+F 5 " 150060RS75000 " H 6500 3500 50  0001 C CNN "Part"
+	1    6500 3500
+	1    0    0    -1
+$EndComp
+Text Notes 6400 5200 0    50   ~ 0
+Upgrades:\n- use LVC1G10 (3 input nand) and evaluate\n  LEG# with additional input/jumper\n- add USB mux option (e.g. TS3USB221)
 $EndSCHEMATC

Commit message: more part numbers
Parts:
- D1101, D1102: Part 150060GS75000 -> 150060GS75000
- D1103: Part 150060RS75000 -> 150060RS75000
- FL1101, FL1102: Manufacturer (none) -> Wurth; Part (none) -> 744231371
- J1101: Manufacturer (none) -> Molex; Part (none) -> 473460001
- J1102: Manufacturer (none) -> GCT; Part (none) -> USB4085
- L1101: Manufacturer TOKO -> Sumida; Model FDV0530S-1R0 -> (none); Part (none) -> CDMC6D28NP-1R0MC
Changed lines of the file:
@@
 F 2 "Connector_USB:USB_Micro-B_Molex_47346-0001" H 1150 6350 50  0001 C CNN
 F 3 " ~" H 1150 6350 50  0001 C CNN
+F 4 "Molex" H 1000 6400 50  0001 C CNN "Manufacturer"
+F 5 "473460001" H 1000 6400 50  0001 C CNN "Part"
 	1    1000 6400
 	1    0    0    -1
@@
 F 2 "proj_footprints:WE_CNSW" V 1600 7540 50  0001 C CNN
 F 3 "https://www.digikey.com/catalog/en/partgroup/we-cnsw-we-cnsw-hf/22783?mpart=744231371&vendor=732" H 1600 7687 50  0001 C CNN
+F 4 "744231371" H 1600 7500 50  0001 C CNN "Part"
+F 5 "Wurth" H 1600 7500 50  0001 C CNN "Manufacturer"
 	1    1600 7500
 	1    0    0    1
@@
 F 2 "proj_footprints:WE_CNSW" V 1850 6490 50  0001 C CNN
 F 3 "https://www.digikey.com/catalog/en/partgroup/we-cnsw-we-cnsw-hf/22783?mpart=744231371&vendor=732" H 1850 6637 50  0001 C CNN
+F 4 "744231371" H 1850 6450 50  0001 C CNN "Part"
+F 5 "Wurth" H 1850 6450 50  0001 C CNN "Manufacturer"
 	1    1850 6450
 	1    0    0    -1
@@
 F 2 "proj_footprints:L_CDMC6D28" H 6800 1000 50  0001 C CNN
 F 3 "~" H 6800 1000 50  0001 C CNN
-F 4 "TOKO" V 6800 1000 50  0001 C CNN "Manufacturer"
-F 5 "FDV0530S-1R0" V 6800 1000 50  0001 C CNN "Model"
+F 4 "Sumida" V 6800 1000 50  0001 C CNN "Manufacturer"
+F 5 "CDMC6D28NP-1R0MC " V 6800 1000 50  0001 C CNN "Part"
 	1    6800 1000
 	0    1    1    0
@@
 F 3 "~" H 5000 4550 50  0001 C CNN
 F 4 "Wurth" H 5000 4550 50  0001 C CNN "Manufacturer"
-F 5 " 150060GS75000 " H 5000 4550 50  0001 C CNN "Part"
+F 5 "150060GS75000" H 5000 4550 50  0001 C CNN "Part"
 	1    5000 4550
 	0    -1   -1   0
@@
 F 3 "~" H 5350 4550 50  0001 C CNN
 F 4 "Wurth" H 5350 4550 50  0001 C CNN "Manufacturer"
-F 5 " 150060GS75000 " H 5350 4550 50  0001 C CNN "Part"
+F 5 "150060GS75000" H 5350 4550 50  0001 C CNN "Part"
 	1    5350 4550
 	0    -1   -1   0
@@
 F 2 "proj_footprints:USB_C_Receptacle_GCT_USB4085_smaller_holes" H 2250 2100 50  0001 C CNN
 F 3 "https://www.usb.org/sites/default/files/documents/usb_type-c.zip" H 2250 2100 50  0001 C CNN
+F 4 "GCT" H 2100 2100 50  0001 C CNN "Manufacturer"
+F 5 "USB4085" H 2100 2100 50  0001 C CNN "Part"
 	1    2100 2100
 	1    0    0    -1
@@
 F 3 "~" H 6500 3500 50  0001 C CNN
 F 4 "Wurth" H 6500 3500 50  0001 C CNN "Manufacturer"
-F 5 " 150060RS75000 " H 6500 3500 50  0001 C CNN "Part"
+F 5 "150060RS75000" H 6500 3500 50  0001 C CNN "Part"
 	1    6500 3500
 	1    0    0    -1

Commit message: changed inductor to TDK part (availability)
Parts:
- L1101: footprint proj_footprints:L_CDMC6D28 -> proj_footprints:L_TDK_SPM6530; Manufacturer Sumida -> TDK; Part CDMC6D28NP-1R0MC -> SPM6530T-1R0M120
Changed lines of the file:
@@
 F 0 "L1101" V 6622 1000 50  0000 C CNN
 F 1 "1uH" V 6713 1000 50  0000 C CNN
-F 2 "proj_footprints:L_CDMC6D28" H 6800 1000 50  0001 C CNN
+F 2 "proj_footprints:L_TDK_SPM6530" H 6800 1000 50  0001 C CNN
 F 3 "~" H 6800 1000 50  0001 C CNN
-F 4 "Sumida" V 6800 1000 50  0001 C CNN "Manufacturer"
-F 5 "CDMC6D28NP-1R0MC " V 6800 1000 50  0001 C CNN "Part"
+F 4 "TDK" V 6800 1000 50  0001 C CNN "Manufacturer"
+F 5 "SPM6530T-1R0M120" V 6800 1000 50  0001 C CNN "Part"
 	1    6800 1000
 	0    1    1    0

Commit message: don't recall changes...
Parts:
- removed U1103: FT232RL, Package_SO:SSOP-28_5.3x10.2mm_P0.65mm, symbol Interface_USB:FT232RL
- added U1103: FT231XS, Package_SO:SSOP-20_3.9x8.7mm_P0.635mm, symbol Interface_USB:FT231XS
- J1101: value USB_miniB -> USB_microB; footprint Connector_USB:USB_Micro-B_Molex_47346-0001 -> Connector_USB:USB_Micro-B_Molex-105017-0001; Part 473460001 -> 1050170001
- R1113, R1114, R1118: value 1k5 -> 1k; symbol trigbox:R100k -> Device:R_Small
Connections:
- wire segments 136 -> 141
- no-connect marks 23 -> 20
Other:
- moved on the sheet: C1101, R1110
Changed lines of the file:
@@
 $EndDescr
-$Comp
-L Interface_USB:FT232RL U1103
-U 1 1 5C383A94
-P 5400 6800
-F 0 "U1103" H 5750 7750 50  0000 C CNN
-F 1 "FT232RL" H 4950 7750 50  0000 C CNN
-F 2 "Package_SO:SSOP-28_5.3x10.2mm_P0.65mm" H 5400 6800 50  0001 C CNN
-F 3 "http://www.ftdichip.com/Products/ICs/FT232RL.htm" H 5400 6800 50  0001 C CNN
-	1    5400 6800
-	1    0    0    -1
-$EndComp
 $Comp
 L power:GND #PWR?
@@
 	1    0    0    -1
 $EndComp
-Wire Wire Line
-	4600 7500 4600 7800
-Wire Wire Line
-	4600 7800 4750 7800
-Connection ~ 5200 7800
-Wire Wire Line
-	5200 7800 5400 7800
-Connection ~ 5400 7800
-Wire Wire Line
-	5400 7800 5500 7800
-Connection ~ 5500 7800
-Wire Wire Line
-	5500 7800 5600 7800
 Connection ~ 4750 7800
-Wire Wire Line
-	4750 7800 5200 7800
-NoConn ~ 4600 7200
-NoConn ~ 4600 7000
 $Comp
 L fmc:100nF_603 C1101
 U 1 1 5C383AAF
-P 4100 7350
-F 0 "C1101" H 3900 7450 50  0000 L CNN
-F 1 "100nF_603" H 3550 7300 50  0000 L CNN
-F 2 "Capacitor_SMD:C_0603_1608Metric" H 4138 7200 50  0001 C CNN
-F 3 "~" H 4100 7350 50  0001 C CNN
-F 4 "GCJ188R71E104KA12D" H 4225 7550 50  0001 C CNN "Part"
-F 5 "Murata" H 4325 7650 50  0001 C CNN "Manufacturer"
-	1    4100 7350
-	1    0    0    -1
-$EndComp
-Connection ~ 4600 7500
-Wire Wire Line
-	4600 6100 4100 6100
-Wire Wire Line
-	4100 6100 4100 7200
+P 4550 7550
+F 0 "C1101" V 4450 7650 50  0000 L CNN
+F 1 "100nF_603" H 4600 7450 50  0000 L CNN
+F 2 "Capacitor_SMD:C_0603_1608Metric" H 4588 7400 50  0001 C CNN
+F 3 "~" H 4550 7550 50  0001 C CNN
+F 4 "GCJ188R71E104KA12D" H 4675 7750 50  0001 C CNN "Part"
+F 5 "Murata" H 4775 7850 50  0001 C CNN "Manufacturer"
+	1    4550 7550
+	1    0    0    -1
+$EndComp
 Wire Wire Line
 	4600 6800 4300 6800
 Wire Wire Line
-	4300 6800 4300 7300
+	4300 6800 4300 7450
 $Comp
 L power-test-module-rescue:+3V3 #PWR?
 U 1 1 5C383ABB
-P 5300 5800
+P 5400 5850
 AR Path="/5BE73D36/5C383ABB" Ref="#PWR?"  Part="1"
 AR Path="/5C1147CA/5C383ABB" Ref="#PWR?"  Part="1"
@@
 AR Path="/5C4CE703/5C383ABB" Ref="#PWR?"  Part="1"
 AR Path="/60DAA393/5C4CE703/5C383ABB" Ref="#PWR?"  Part="1"
-F 0 "#PWR?" H 5300 5650 50  0001 C CNN
-F 1 "+3V3" H 5315 5973 50  0000 C CNN
-F 2 "" H 5300 5800 50  0001 C CNN
-F 3 "" H 5300 5800 50  0001 C CNN
-	1    5300 5800
+F 0 "#PWR?" H 5400 5700 50  0001 C CNN
+F 1 "+3V3" H 5415 6023 50  0000 C CNN
+F 2 "" H 5400 5850 50  0001 C CNN
+F 3 "" H 5400 5850 50  0001 C CNN
+	1    5400 5850
 	1    0    0    -1
 $EndComp
@@
 L power-test-module-rescue:+5V #PWR?
 U 1 1 5C383AC1
-P 5500 5800
-F 0 "#PWR?" H 5500 5650 50  0001 C CNN
-F 1 "+5V" H 5515 5973 50  0000 C CNN
-F 2 "" H 5500 5800 50  0001 C CNN
-F 3 "" H 5500 5800 50  0001 C CNN
-	1    5500 5800
+P 5200 5850
+F 0 "#PWR?" H 5200 5700 50  0001 C CNN
+F 1 "+5V" H 5215 6023 50  0000 C CNN
+F 2 "" H 5200 5850 50  0001 C CNN
+F 3 "" H 5200 5850 50  0001 C CNN
+	1    5200 5850
 	1    0    0    -1
 $EndComp
@@
 P 1000 6400
 F 0 "J1101" H 1055 6867 50  0000 C CNN
-F 1 "USB_miniB" H 1000 6800 50  0000 C CNN
-F 2 "Connector_USB:USB_Micro-B_Molex_47346-0001" H 1150 6350 50  0001 C CNN
+F 1 "USB_microB" H 1000 6800 50  0000 C CNN
+F 2 "Connector_USB:USB_Micro-B_Molex-105017-0001" H 1150 6350 50  0001 C CNN
 F 3 " ~" H 1150 6350 50  0001 C CNN
 F 4 "Molex" H 1000 6400 50  0001 C CNN "Manufacturer"
-F 5 "473460001" H 1000 6400 50  0001 C CNN "Part"
+F 5 "1050170001" H 1000 6400 50  0001 C CNN "Part"
 	1    1000 6400
 	1    0    0    -1
 $EndComp
 NoConn ~ 1300 6600
-Wire Wire Line
-	4300 6200 4300 6600
 $Comp
 L power:GND #PWR?
@@
 	1    0    0    1
 $EndComp
-Wire Wire Line
-	4100 7500 4300 7500
 $Comp
 L trigbox:R10k R1111
 U 1 1 5C383AE5
-P 4300 7400
-F 0 "R1111" H 4359 7430 50  0000 L CNN
-F 1 "10k" H 4359 7354 30  0000 L CNN
-F 2 "Resistor_SMD:R_0603_1608Metric" H 4300 7400 50  0001 C CNN
-F 3 "~" H 4300 7400 50  0001 C CNN
-	1    4300 7400
-	1    0    0    -1
-$EndComp
-Connection ~ 4300 7500
-Wire Wire Line
-	4300 7500 4600 7500
-$Comp
-L Device:R_Small R1110
-U 1 1 5C383AEE
-P 4300 6700
-F 0 "R1110" H 4359 6730 50  0000 L CNN
-F 1 "5k1" H 4359 6654 30  0000 L CNN
-F 2 "Resistor_SMD:R_0603_1608Metric" H 4300 6700 50  0001 C CNN
-F 3 "~" H 4300 6700 50  0001 C CNN
-	1    4300 6700
-	1    0    0    -1
-$EndComp
-Connection ~ 4300 6800
+P 4300 7550
+F 0 "R1111" H 4359 7580 50  0000 L CNN
+F 1 "10k" H 4359 7504 30  0000 L CNN
+F 2 "Resistor_SMD:R_0603_1608Metric" H 4300 7550 50  0001 C CNN
+F 3 "~" H 4300 7550 50  0001 C CNN
+	1    4300 7550
+	-1   0    0    -1
+$EndComp
 $Comp
 L power:PWR_FLAG #FLG?
@@
 	1    0    0    -1
 $EndComp
-NoConn ~ 6200 6300
-NoConn ~ 6200 6500
-NoConn ~ 6200 7100
-NoConn ~ 6200 7200
-NoConn ~ 6200 7300
-NoConn ~ 6200 7400
-NoConn ~ 6200 7500
-NoConn ~ 6200 6400
-NoConn ~ 6200 6600
-NoConn ~ 6200 6700
-NoConn ~ 6200 6800
+NoConn ~ 6000 6400
+NoConn ~ 6000 6600
+NoConn ~ 6000 7100
+NoConn ~ 6000 7200
+NoConn ~ 6000 7300
+NoConn ~ 6000 7400
+NoConn ~ 6000 6500
+NoConn ~ 6000 6700
+NoConn ~ 6000 6800
+NoConn ~ 6000 6900
 $Comp
 L Interface_USB:USB3740B-AI9 U1101
@@
 $EndComp
 Wire Wire Line
-	4600 6400 3150 6400
-Wire Wire Line
 	4600 6500 3150 6500
 $Comp
@@
 Wire Wire Line
 	3300 6100 3300 6200
-Wire Wire Line
-	3300 6200 4300 6200
 $Comp
 L power-test-module-rescue:+5V #PWR?
@@
 AR Path="/5C4CE703/5C3CF1BE" Ref="R1109"  Part="1"
 AR Path="/60DAA393/5C4CE703/5C3CF1BE" Ref="R1109"  Part="1"
-F 0 "R1109" H 4100 5400 50  0000 L CNN
+F 0 "R1109" H 4000 5400 50  0000 L CNN
 F 1 "5k1" H 4100 5300 50  0000 L CNN
 F 2 "Resistor_SMD:R_0603_1608Metric" H 4300 5350 50  0001 C CNN
@@
 AR Path="/5C4CE703/5C3CF1CB" Ref="R1112"  Part="1"
 AR Path="/60DAA393/5C4CE703/5C3CF1CB" Ref="R1112"  Part="1"
-F 0 "R1112" H 4300 5250 50  0000 L CNN
+F 0 "R1112" H 4200 5250 50  0000 L CNN
 F 1 "35k7" H 4250 5150 50  0000 L CNN
 F 2 "Resistor_SMD:R_0603_1608Metric" H 4500 5200 50  0001 C CNN
@@
 	5350 4800 4000 4800
 $Comp
-L trigbox:R100k R?
+L Device:R_Small R?
 U 1 1 5C417A62
 P 5000 4300
@@
 AR Path="/5C4CE703/5C417A62" Ref="R1113"  Part="1"
 AR Path="/60DAA393/5C4CE703/5C417A62" Ref="R1113"  Part="1"
-F 0 "R1113" H 4800 4350 50  0000 L CNN
-F 1 "1k5" H 4800 4250 30  0000 L CNN
+F 0 "R1113" H 4750 4450 50  0000 L CNN
+F 1 "1k" H 4800 4250 30  0000 L CNN
 F 2 "Resistor_SMD:R_0603_1608Metric" H 5000 4300 50  0001 C CNN
 F 3 "~" H 5000 4300 50  0001 C CNN
@@
 $EndComp
 $Comp
-L trigbox:R100k R?
+L Device:R_Small R?
 U 1 1 5C417B66
 P 5350 4300
@@
 AR Path="/5C4CE703/5C417B66" Ref="R1114"  Part="1"
 AR Path="/60DAA393/5C4CE703/5C417B66" Ref="R1114"  Part="1"
-F 0 "R1114" H 5150 4350 50  0000 L CNN
-F 1 "1k5" H 5150 4250 30  0000 L CNN
+F 0 "R1114" H 5050 4450 50  0000 L CNN
+F 1 "1k" H 5150 4250 30  0000 L CNN
 F 2 "Resistor_SMD:R_0603_1608Metric" H 5350 4300 50  0001 C CNN
 F 3 "~" H 5350 4300 50  0001 C CNN
@@
 $EndComp
 $Comp
-L trigbox:R100k R?
+L Device:R_Small R?
 U 1 1 5C417BFB
 P 6850 3400
@@
 AR Path="/5C4CE703/5C417BFB" Ref="R1118"  Part="1"
 AR Path="/60DAA393/5C4CE703/5C417BFB" Ref="R1118"  Part="1"
-F 0 "R1118" H 6650 3450 50  0000 L CNN
-F 1 "1k5" H 6650 3350 30  0000 L CNN
+F 0 "R1118" H 6950 3450 50  0000 L CNN
+F 1 "1k" H 6650 3350 30  0000 L CNN
 F 2 "Resistor_SMD:R_0603_1608Metric" H 6850 3400 50  0001 C CNN
 F 3 "~" H 6850 3400 50  0001 C CNN
@@
 $EndComp
 Wire Wire Line
-	6200 6100 6550 6100
-Wire Wire Line
-	6200 6200 6550 6200
+	6000 6200 6350 6200
+Wire Wire Line
+	6000 6300 6350 6300
 Wire Wire Line
 	5700 2150 5700 2700
@@
 Text Label 2150 5250 0    50   ~ 0
 USB_C_D_N
-Text HLabel 6550 6100 2    50   Output ~ 0
+Text HLabel 6350 6200 2    50   Output ~ 0
 UART_TX_OUT
-Text HLabel 6550 6200 2    50   Input ~ 0
+Text HLabel 6350 6300 2    50   Input ~ 0
 UART_RX_IN
 $Comp
@@
 Text Notes 6400 5200 0    50   ~ 0
 Upgrades:\n- use LVC1G10 (3 input nand) and evaluate\n  LEG# with additional input/jumper\n- add USB mux option (e.g. TS3USB221)
+$Comp
+L Interface_USB:FT231XS U1103
+U 1 1 60F229DF
+P 5300 6800
+F 0 "U1103" H 5650 7650 50  0000 C CNN
+F 1 "FT231XS" H 4700 7650 50  0000 C CNN
+F 2 "Package_SO:SSOP-20_3.9x8.7mm_P0.635mm" H 6300 6000 50  0001 C CNN
+F 3 "https://www.ftdichip.com/Support/Documents/DataSheets/ICs/DS_FT231X.pdf" H 5300 6800 50  0001 C CNN
+	1    5300 6800
+	1    0    0    -1
+$EndComp
+$Comp
+L Device:R_Small R1110
+U 1 1 5C383AEE
+P 3700 6200
+F 0 "R1110" V 3800 6000 50  0000 L CNN
+F 1 "5k1" V 3800 6300 30  0000 L CNN
+F 2 "Resistor_SMD:R_0603_1608Metric" H 3700 6200 50  0001 C CNN
+F 3 "~" H 3700 6200 50  0001 C CNN
+	1    3700 6200
+	0    -1   -1   0
+$EndComp
+Wire Wire Line
+	3300 6200 3600 6200
+Wire Wire Line
+	4750 7800 5200 7800
+Wire Wire Line
+	3800 6200 4300 6200
+Wire Wire Line
+	4300 6200 4300 6800
+Connection ~ 4300 6800
+Wire Wire Line
+	4550 6200 4600 6200
+Wire Wire Line
+	4550 6200 4550 7400
+Wire Wire Line
+	4600 6600 3900 6600
+Wire Wire Line
+	3900 6600 3900 6400
+Wire Wire Line
+	3900 6400 3150 6400
+Wire Wire Line
+	4300 7650 4300 7800
+Wire Wire Line
+	4300 7800 4550 7800
+Wire Wire Line
+	4550 7700 4550 7800
+Connection ~ 4550 7800
+Wire Wire Line
+	4550 7800 4750 7800
+Wire Wire Line
+	5200 7700 5200 7800
+Connection ~ 5200 7800
+Wire Wire Line
+	5200 7800 5400 7800
+Wire Wire Line
+	5400 7700 5400 7800
+Wire Wire Line
+	5200 5850 5200 5900
+Wire Wire Line
+	5400 5850 5400 5900
 $EndSCHEMATC
