File: power-test-module.kicad_pcb (KiCad board)
At the start: 2 copper layers, 38.4 x 23.9 mm, 42 parts, among them J1001 Conn_02x06_Odd_Even, J1002 USB_miniB, J1003 USB_C_Receptacle_USB2.0, U1001 USB3740B-AI9, U1002 UTC2000, U1003 FT232RL, U1004 74LVC1G00, U1005 SC185

Commit message: removed global labels for UART-TX/RX
There referred to MIO pins on the CPU board which don't really
belong here; also: avoid global labels for a module.
Connections:
- net UART_RX_MIO14 renamed /UART_TX_OUT
- net UART_TX_MIO15 renamed /UART_RX_IN

Commit message: re-annotated for merging; updated PCB
Parts:
- removed J1001: Conn_02x06_Odd_Even, Connector_PinHeader_2.54mm:PinHeader_2x06_P2.54mm_Vertical
- renumbered C1001 to C1101, C1002 to C1102, C1003 to C1103, C1004 to C1104, C1005 to C1105, C1006 to C1106, C1007 to C1107, C1008 to C1108, D1001 to D1101, D1002 to D1102, D1003 to D1103, FL1001 to FL1101, FL1002 to FL1102, J1002 to J1101, J1003 to J1102, JP1001 to JP1101, JP1002 to JP1102, L1001 to L1101, R1001 to R1101, R1002 to R1102, R1003 to R1103, R1004 to R1104, R1005 to R1105, R1006 to R1106, R1007 to R1107, R1008 to R1108, R1009 to R1109, R1010 to R1110, R1011 to R1111, R1012 to R1112, R1013 to R1113, R1014 to R1114, R1015 to R1115, R1016 to R1116, R1017 to R1117, R1018 to R1118, U1001 to U1101, U1002 to U1102, U1003 to U1103, U1004 to U1104, U1005 to U1105
